Commit message: 土台等のサイズ修正

File: Assets/Urdf/robot_arm2.urdf (robot description, URDF)
Before this commit: robot robot_arm, 4 links, 3 joints
Links:
- link base_link: geometry collision box size=0.2 0.2 0.05; visual box size=0.2 0.2 0.05
- link torso: geometry collision cylinder length=0.5 radius=0.05; visual cylinder length=0.5 radius=0.05
- link upper_arm: geometry collision cylinder length=0.4 radius=0.05; visual cylinder length=0.4 radius=0.05
Joints:
- joint hip: origin xyz=0.0 0.0 0.1 rpy=0 0 0 -> xyz=0.0 0.0 0.05 rpy=0 0 0
- joint shoulder: origin xyz=0.0 -0.2 2.3 rpy=0 0 0 -> xyz=0.0 -0.1 0.45 rpy=0 0 0
