Commit message: ロボットアーム追加

File: Assets/Urdf/robot_arm.urdf (robot description, URDF)
Before this commit: robot robot_arm, 4 links, 3 joints
Links:
- added link lower_arm, mass 1.0; collision cylinder length=2.5 radius=0.1; visual cylinder length=2.5 radius=0.1
- link torso: geometry collision cylinder length=0.2 radius=0.1; visual cylinder length=0.2 radius=0.1
- link upper_arm: geometry collision cylinder length=2.5 radius=0.1; visual cylinder length=2.5 radius=0.1
Joints:
- added joint elbow: type revolute, parent lower_arm, child upper_arm, origin xyz=0.0 0.2 2.35 rpy=0 0 0, axis 0 1 0, limit lower=-0.00 upper=2.00 effort=0.5293 velocity=6.159937255
- joint shoulder: child upper_arm -> lower_arm; origin xyz=0.0 -0.2 2.3 rpy=0 0 0 -> xyz=0.0 -0.2 0.1 rpy=0 0 0

Commit message: ArmRobotの修正

File: Assets/Urdf/robot_arm.urdf (robot description, URDF)
Before this commit: robot robot_arm, 5 links, 4 joints
Links:
- added link hand, mass 1.0; collision cylinder length=0.2 radius=0.1; visual cylinder length=0.2 radius=0.1
- added link on_hand, mass 1.0; collision box size=0.4 0.4 0.1; visual box size=0.4 0.4 0.1
Joints:
- added joint on_hand: type revolute, parent hand, child on_hand, origin xyz=0.0 0.0 0.2 rpy=0 0 0, axis 0 1 0, limit lower=0.00 upper=0.00 effort=0.5293 velocity=6.159937255
- added joint wrist: type revolute, parent upper_arm, child hand, origin xyz=0.0 -0.2 2.4 rpy=0 0 0, axis 0 1 0, limit lower=0.00 upper=0.00 effort=0.5293 velocity=6.159937255
- joint elbow: limit lower=-0.00 upper=2.00 effort=0.5293 velocity=6.159937255 -> lower=0.00 upper=2.00 effort=0.5293 velocity=6.159937255
- joint hip: limit lower=-1.00 upper=0.00 effort=0.5293 velocity=6.159937255 -> lower=0.00 upper=0.00 effort=0.5293 velocity=6.159937255
- joint shoulder: limit lower=-0.00 upper=2.00 effort=0.5293 velocity=6.159937255 -> lower=-1.00 upper=0.00 effort=0.5293 velocity=6.159937255

Commit message: アームロボット　MoveIt

File: Assets/Urdf/robot_arm.urdf (robot description, URDF)
Before this commit: robot robot_arm, 5 links, 4 joints
Joints:
- joint hip: limit lower=-1.00 upper=0.00 effort=0.5293 velocity=6.159937255 -> lower=-0.00 upper=0.00 effort=0.5293 velocity=6.159937255
- joint shoulder: limit lower=-0.00 upper=2.00 effort=0.5293 velocity=6.159937255 -> lower=-1.00 upper=0.00 effort=0.5293 velocity=6.159937255

Commit message: アームロボットの変更とサブスクライブ設定

File: Assets/Urdf/robot_arm.urdf (robot description, URDF)
Before this commit: robot robot_arm, 7 links, 6 joints
Links:
- removed link on_hand
- added link parm, mass 1.0; collision box size=0.4 0.4 0.1; visual box size=0.4 0.4 0.1
Joints:
- joint on_hand: child on_hand -> parm
- joint wrist: limit lower=0.00 upper=0.00 effort=0.5293 velocity=6.159937255 -> lower=-1.00 upper=0.00 effort=0.5293 velocity=6.159937255
