Commit message: mobile_robotのGUI自走走行

File: Assets/Urdf/mobile_robot.urdf (robot description, URDF)
Before this commit: robot mobile_robot, 6 links, 5 joints
Links:
- removed link base_footprint
- added link sensor_link, mass 1e-5; collision box size=0.1 0.1 0.1; visual box size=0.1 0.1 0.1
Joints:
- removed joint base_joint
- added joint sensor_joint: type fixed, parent base_link, child sensor_link, origin xyz=0 0 0.2 rpy=0 0 0, axis 0 1 0

Commit message: 移動ロボットの修正とマップ作成

File: Assets/Urdf/mobile_robot.urdf (robot description, URDF)
Before this commit: robot mobile_robot, 6 links, 5 joints
Links:
- removed link sensor_link
- added link base_scan, mass 1e-5; collision box size=0.1 0.1 0.1; visual box size=0.1 0.1 0.1
Joints:
- joint sensor_joint: child sensor_link -> base_scan

Commit message: スクリプトを用いて移動ロボットを動かす

File: Assets/Urdf/mobile_robot.urdf (robot description, URDF)
Before this commit: robot mobile_robot, 6 links, 5 joints
Links:
- added link base_footprint
Joints:
- removed joint sensor_joint
- added joint base_joint: type fixed, parent base_footprint, child base_link, origin xyz=0 0 0.126
- added joint scan_joint: type fixed, parent base_link, child base_scan, origin xyz=0 0 0.2 rpy=0 0 0, axis 0 1 0
